File: Interface_DAC/Interface_DAC.kicad_pcb (KiCad board)
At the start: 4 copper layers, 68 x 45 mm, 122 parts, among them J1 Barrel_Jack_Switch_Pin3Ring, J2 Conn_Coaxial, J3 USB_C_Receptacle_USB2.0_16P, Q1 AO3401, SW1 SW_Push, SW2 SW_DIP_x02, U1 MIMXRT1011DAE5A, U10 TPS7A3301RGW, U2 W25Q32JVUU, U3 UM803RS, U4 PCM1794A, U5 TUSB320, U6 SN74LVC2G14DBV, U7 TPS62A02ADRL, U8 TPS65131RGE, U9 TPS7A4701xRGW, Y1 KC2520Z, Y2 KC2520Z, Y3 24M

Commit message: Schematic Tinkering and PCB Layout
Parts:
- added C40: 4.7n, Capacitor_SMD:C_0402_1005Metric, F.Cu at (85.2, 72.0)
- added C43: 10n, Capacitor_SMD:C_0402_1005Metric, F.Cu at (91.5, 69.2)
- added C49: 10n, Capacitor_SMD:C_0402_1005Metric, F.Cu at (90.0, 68.7)
- added C50: 4.7n, Capacitor_SMD:C_0402_1005Metric, F.Cu at (85.8, 66.7)
- added C53: 4.7n, Capacitor_SMD:C_0402_1005Metric, F.Cu at (85.2, 80.3)
- added C54: 10n, Capacitor_SMD:C_0402_1005Metric, F.Cu at (91.5, 77.8)
- added C55: 10n, Capacitor_SMD:C_0402_1005Metric, F.Cu at (90.0, 78.3)
- added C56: 4.7n, Capacitor_SMD:C_0402_1005Metric, F.Cu at (85.8, 75.0)
- added R13: 820, Resistor_SMD:R_0402_1005Metric, F.Cu at (85.2, 81.3)
- added R14: 240, Resistor_SMD:R_0402_1005Metric, F.Cu at (91.5, 78.8)
- added R17: 510, Resistor_SMD:R_0402_1005Metric, F.Cu at (86.8, 80.8)
- added R18: 510, Resistor_SMD:R_0402_1005Metric, F.Cu at (87.2, 74.5)
- added R19: 240, Resistor_SMD:R_0402_1005Metric, F.Cu at (89.0, 78.3)
- added R2: 2.2M, Resistor_SMD:R_0402_1005Metric, F.Cu at (54.0, 54.3)
- added R20: 820, Resistor_SMD:R_0402_1005Metric, F.Cu at (85.8, 74.0)
- added R3: 820, Resistor_SMD:R_0402_1005Metric, F.Cu at (85.2, 73.0)
- added R4: 240, Resistor_SMD:R_0402_1005Metric, F.Cu at (91.5, 68.2)
- added R5: 510, Resistor_SMD:R_0402_1005Metric, F.Cu at (86.8, 72.5)
- added R6: 510, Resistor_SMD:R_0402_1005Metric, F.Cu at (87.2, 66.2)
- added R7: 240, Resistor_SMD:R_0402_1005Metric, F.Cu at (89.0, 68.7)
- added R8: 820, Resistor_SMD:R_0402_1005Metric, F.Cu at (85.8, 65.7)
- added U4: OPA1612AxD, Package_SON:WSON-8-1EP_3x3mm_P0.5mm_EP1.2x2mm_ThermalVias, F.Cu at (85.2, 69.3)
- added U5: OPA1612AxD, Package_SO:SOIC-8_3.9x4.9mm_P1.27mm, F.Cu at (90.5, 73.5)
- added U6: OPA1612AxD, Package_SON:WSON-8-1EP_3x3mm_P0.5mm_EP1.2x2mm_ThermalVias, F.Cu at (85.2, 77.7)
- moved Y1 117.7 mm to (73.5, 65.0)
- moved Y2 116.7 mm to (78.5, 65.0)
- moved C25 109.3 mm to (73.5, 67.2), turned to 180 degrees
- moved C20 107.5 mm to (75.5, 64.5), turned to -90 degrees
- moved C26 104.8 mm to (78.5, 67.2), turned to 180 degrees
- moved C21 103.7 mm to (80.5, 64.5), turned to -90 degrees
- moved C69 75.8 mm to (69.3, 53.8), turned to 180 degrees
- moved L3 75.7 mm to (71.1, 59.9)
- moved C58 75.5 mm to (71.5, 51.3)
- moved C62 75.5 mm to (74.5, 51.3)
- moved C67 75.5 mm to (77.8, 56.6)
- moved D4 75.5 mm to (76.8, 54.2)
- moved L5 75.5 mm to (78.8, 54.2)
- moved R22 75.5 mm to (72.5, 51.3)
- moved R25 75.5 mm to (73.5, 51.3)
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- renumbered C40 to C41, C41 to C42, C42 to C44, C43 to C45, C44 to C46, C45 to C47, C46 to C48, C47 to C51, C48 to C52, C49 to C57, C50 to C58, C51 to C59, C52 to C60, C53 to C61, C54 to C62, C55 to C63, C56 to C64, C57 to C65, C58 to C66, C59 to C67, C60 to C68, C61 to C69, C62 to C70, C63 to C71, C64 to C72, C65 to C73, C66 to C74, C67 to C75, C68 to C76, C69 to C77, R3 to R10, R4 to R11, R5 to R12, R6 to R15, R7 to R16, R8 to R21, R9 to R22, R10 to R23, R11 to R24, R12 to R25, R13 to R26, R14 to R27, R15 to R28, R16 to R29, R17 to R30, R18 to R31, R19 to R32, R2 to R9, U7 to U10, U8 to U11, U9 to U12, U10 to U13, U4 to U7, U5 to U8, U6 to U9
Connections:
- U13 pad 10: GND -> (no net)
- U13 pad 11: GND -> (no net)
- U13 pad 12: GND -> (no net)
- U13 pad 17: GND -> (no net)
- U13 pad 18: GND -> (no net)
- U13 pad 19: GND -> (no net)
- U13 pad 2: -9VA -> (no net)
- U13 pad 4: GND -> (no net)
- U13 pad 5: GND -> (no net)
- U13 pad 6: GND -> (no net)
- U13 pad 8: GND -> (no net)
- U13 pad 9: GND -> (no net)
- U7 pad 17: unconnected-(U4-IOUTR+-Pad17) -> IOUTRP
- U7 pad 18: unconnected-(U4-IOUTR--Pad18) -> IOUTRN
- U7 pad 25: unconnected-(U4-IOUTL+-Pad25) -> IOUTLP
- U7 pad 26: unconnected-(U4-IOUTL--Pad26) -> IOUTLN
Routing:
- net Net-(U11-FBP): track 0.00 -> 3.35 mm
- net GND: track 61.0 -> 64.0 mm, vias 1 -> 6
- net I2S_LRCK: track 9.47 -> 6.71 mm
- net Net-(U1A-VDD_HIGH_CAP): track 2.70 -> 0.00 mm
- net Net-(U11-ENN): track 0.00 -> 2.29 mm
- net I2S_BCK: track 7.69 -> 5.59 mm
- net Net-(U11-CP): track 0.00 -> 1.81 mm
- net Net-(U11-CN): track 0.00 -> 1.76 mm
- net I2S_SCK: track 7.23 -> 5.59 mm
- net Net-(U1B-XTALI): track 7.23 -> 8.67 mm
- net I2S_DATA: track 7.20 -> 6.39 mm
- net Net-(U7-BCK): track 3.11 -> 2.33 mm
- net Net-(U7-LRCK): track 3.40 -> 2.62 mm
- net Net-(U7-DATA): track 3.26 -> 2.48 mm
- net Net-(U7-SCK): track 2.97 -> 2.19 mm
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- added copper zone on F.Cu, net +10V
- added copper zone on F.Cu, net Net-(D3-A)
- added copper zone on F.Cu, net Net-(Q1-D)
